File: pcb/pcb.kicad_sch (KiCad schematic)
At the start: 0 parts

Commit message: second update
Parts:
- added D1, D10, D11, D12, D13, D14, D15, D16, D17, D18, D19, D2, D20, D21, D22, D23, D24, D25, D26, D27, D28, D29, D3, D30, D31, D32, D33, D34, D35, D36, D37, D38, D39, D4, D40, D41, D42, D43, D44, D45, D46, D47, D48, D49, D5, D50, D51, D52, D53, D54, D55, D56, D57, D58, D59, D6, D60, D61, D62, D63, D64, D65, D66, D67, D68, D69, D7, D70, D71, D72, D73, D74, D75, D76, D77, D78, D79, D8, D80, D81, D82, D83, D9: 1N4148, Diode_THT:D_DO-35_SOD27_P7.62mm_Horizontal, symbol Diode:1N4148
- added SW1, SW10, SW11, SW12, SW13, SW14, SW15, SW16, SW17, SW18, SW19, SW2, SW20, SW21, SW22, SW23, SW24, SW25, SW26, SW27, SW28, SW29, SW3, SW30, SW31, SW32, SW33, SW34, SW35, SW36, SW37, SW38, SW39, SW4, SW40, SW41, SW42, SW43, SW44, SW45, SW46, SW47, SW48, SW49, SW5, SW50, SW51, SW52, SW53, SW54, SW55, SW56, SW57, SW58, SW59, SW6, SW60, SW61, SW62, SW63, SW64, SW65, SW66, SW67, SW68, SW69, SW7, SW70, SW71, SW72, SW73, SW74, SW75, SW76, SW77, SW78, SW79, SW8, SW80, SW81, SW82, SW83, SW9: SW_Push_45deg, symbol Switch:SW_Push_45deg
- added SW84, SW85: SW_Push, symbol Switch:SW_Push
- added SW88: RotaryEncoder, symbol Device:RotaryEncoder
- added U1, U2: nice_nano, symbol nicenano:nice_nano
Connections:
- new net: D79.2 (A), SW79.2
- new net: D67.2 (A), SW67.2
- new net: D13.2 (A), SW13.2
- new net: D39.2 (A), SW39.2
- new net: D81.2 (A), SW81.2
- new net: D54.2 (A), SW54.2
- new net: D60.2 (A), SW60.2
- new net: D18.2 (A), SW18.2
- new net: D63.2 (A), SW63.2
- new net: D28.2 (A), SW28.2
- new net: D47.2 (A), SW47.2
- new net: D6.2 (A), SW6.2
- new net: D19.2 (A), SW19.2
- new net: D10.2 (A), SW10.2
- new net: D4.2 (A), SW4.2
- new net: D26.2 (A), SW26.2
- new net: D41.2 (A), SW41.2
- new net: D53.2 (A), SW53.2
- new net: D15.2 (A), SW15.2
- new net: D75.2 (A), SW75.2
- new net: D64.2 (A), SW64.2
- new net: D43.2 (A), SW43.2
- new net: D35.2 (A), SW35.2
- new net: D24.2 (A), SW24.2
- new net: D73.2 (A), SW73.2
- new net: D57.2 (A), SW57.2
- new net: D70.2 (A), SW70.2
- new net: D76.2 (A), SW76.2
- new net: D59.2 (A), SW59.2
- new net: D78.2 (A), SW78.2
- new net: D9.2 (A), SW9.2
- new net: D34.2 (A), SW34.2
- new net: D2.2 (A), SW2.2
- new net: D8.2 (A), SW8.2
- new net: D42.2 (A), SW42.2
- new net: D56.2 (A), SW56.2
- new net: D52.2 (A), SW52.2
- new net: D71.2 (A), SW71.2
- new net: D46.2 (A), SW46.2
- new net: D33.2 (A), SW33.2
- new net: D38.2 (A), SW38.2
- new net: D83.2 (A), SW83.2
- new net: D30.2 (A), SW30.2
- new net: D68.2 (A), SW68.2
- new net: D25.2 (A), SW25.2
- new net: D80.2 (A), SW80.2
- new net: D14.2 (A), SW14.2
- new net: D1.2 (A), SW1.2
- new net: D17.2 (A), SW17.2
- new net: D20.2 (A), SW20.2
- new net: D36.2 (A), SW36.2
- new net: D45.2 (A), SW45.2
- new net: D29.2 (A), SW29.2
- new net: D48.2 (A), SW48.2
- new net: D31.2 (A), SW31.2
- new net: D3.2 (A), SW3.2
- new net: D12.2 (A), SW12.2
- new net: D55.2 (A), SW55.2
- new net: D77.2 (A), SW77.2
- new net: D49.2 (A), SW49.2
- new net: D22.2 (A), SW22.2
- new net: D51.2 (A), SW51.2
- new net: D23.2 (A), SW23.2
- new net: D37.2 (A), SW37.2
- new net: D21.2 (A), SW21.2
- new net: D5.2 (A), SW5.2
- new net: D58.2 (A), SW58.2
- new net: D69.2 (A), SW69.2
- new net: D74.2 (A), SW74.2
- new net: D44.2 (A), SW44.2
- new net: D32.2 (A), SW32.2
- new net: D82.2 (A), SW82.2
- new net: D27.2 (A), SW27.2
- new net: D72.2 (A), SW72.2
- new net: D7.2 (A), SW7.2
- new net: D65.2 (A), SW65.2
- new net: D40.2 (A), SW40.2
- new net: D61.2 (A), SW61.2
- new net: D16.2 (A), SW16.2
- new net: D66.2 (A), SW66.2
- new net: D11.2 (A), SW11.2
- new net: D50.2 (A), SW50.2
- new net: D62.2 (A), SW62.2
- new net A: SW88.A, U2.17 (P1.15)
- new net B: SW88.B, U2.16 (P1.13)
- new net GND: SW84.2, SW85.2
- new net GND_MCU1: U1.23 (GND)
- new net GND_MCU2: SW88.C, U2.23 (GND)
- new net RST_L: SW84.1, U1.22 (RST)
- new net RST_R: SW85.1, U2.22 (RST)
- new net col_L1: SW1.1, SW15.1, SW22.1, SW28.1, SW34.1, SW8.1, U1.1 (TX0/P0.06)
- new net col_L2: SW16.1, SW2.1, SW23.1, SW29.1, SW35.1, SW9.1, U1.2 (RX1/P0.08)
- new net col_L3: SW10.1, SW17.1, SW24.1, SW3.1, SW30.1, SW36.1, U1.5 (P0.17)
- new net col_L4: SW11.1, SW18.1, SW25.1, SW31.1, SW37.1, SW4.1, U1.6 (P0.20)
- new net col_L5: SW12.1, SW19.1, SW26.1, SW32.1, SW5.1, U1.7 (P0.22)
- new net col_L6: SW13.1, SW20.1, SW27.1, SW33.1, SW6.1, U1.8 (P0.24)
- new net col_L7: SW14.1, SW21.1, SW7.1, U1.9 (P1.00)
- new net col_R1: SW38.1, SW46.1, SW54.1, SW62.1, SW70.1, SW78.1, U2.1 (TX0/P0.06)
- new net col_R2: SW39.1, SW47.1, SW55.1, SW63.1, SW71.1, U2.2 (RX1/P0.08)
- new net col_R3: SW40.1, SW48.1, SW56.1, SW64.1, SW72.1, U2.5 (P0.17)
- new net col_R4: SW41.1, SW49.1, SW57.1, SW65.1, SW73.1, SW79.1, U2.6 (P0.20)
- new net col_R5: SW42.1, SW50.1, SW58.1, SW66.1, SW74.1, SW80.1, U2.7 (P0.22)
- new net col_R6: SW43.1, SW51.1, SW59.1, SW67.1, SW75.1, SW81.1, U2.8 (P0.24)
- new net col_R7: SW44.1, SW52.1, SW60.1, SW68.1, SW76.1, SW82.1, U2.9 (P1.00)
- new net col_R8: SW45.1, SW53.1, SW61.1, SW69.1, SW77.1, SW83.1, U2.10 (P0.11)
- new net row_L1: D1.1 (K), D2.1 (K), D3.1 (K), D4.1 (K), D5.1 (K), D6.1 (K), D7.1 (K), U1.10 (P0.11)
- new net row_L2: D10.1 (K), D11.1 (K), D12.1 (K), D13.1 (K), D14.1 (K), D8.1 (K), D9.1 (K), U1.11 (P1.04)
- new net row_L3: D15.1 (K), D16.1 (K), D17.1 (K), D18.1 (K), D19.1 (K), D20.1 (K), D21.1 (K), U1.12 (P1.06)
- new net row_L4: D22.1 (K), D23.1 (K), D24.1 (K), D25.1 (K), D26.1 (K), D27.1 (K), U1.13 (NFC1/P0.09)
- new net row_L5: D28.1 (K), D29.1 (K), D30.1 (K), D31.1 (K), D32.1 (K), D33.1 (K), U1.14 (NFC2/P0.10)
- new net row_L6: D34.1 (K), D35.1 (K), D36.1 (K), D37.1 (K), U1.15 (P1.11)
- new net row_R1: D38.1 (K), D39.1 (K), D40.1 (K), D41.1 (K), D42.1 (K), D43.1 (K), D44.1 (K), D45.1 (K), U2.11 (P1.04)
- new net row_R2: D46.1 (K), D47.1 (K), D48.1 (K), D49.1 (K), D50.1 (K), D51.1 (K), D52.1 (K), D53.1 (K), U2.12 (P1.06)
- new net row_R3: D54.1 (K), D55.1 (K), D56.1 (K), D57.1 (K), D58.1 (K), D59.1 (K), D60.1 (K), D61.1 (K), U2.13 (NFC1/P0.09)
- new net row_R4: D62.1 (K), D63.1 (K), D64.1 (K), D65.1 (K), D66.1 (K), D67.1 (K), D68.1 (K), D69.1 (K), U2.14 (NFC2/P0.10)
- new net row_R5: D70.1 (K), D71.1 (K), D72.1 (K), D73.1 (K), D74.1 (K), D75.1 (K), D76.1 (K), D77.1 (K), U2.15 (P1.11)
- new net row_R6: D78.1 (K), D79.1 (K), D80.1 (K), D81.1 (K), D82.1 (K), D83.1 (K)
- no-connect marks 0 -> 20
Other:
- added sheet Left Keys (leftkeys.kicad_sch)
- added sheet Left MCU (leftmcu.kicad_sch)
- added sheet Right Keys (rightkeys.kicad_sch)
- added sheet Right MCU (rightmcu.kicad_sch)
