File: pcb/left_split/_autosave-left_split.kicad_sch (KiCad schematic)
At the start: 76 parts, among them SW1 SW_Push_45deg, SW10 SW_Push_45deg, SW11 SW_Push_45deg, SW12 SW_Push_45deg, SW13 SW_Push_45deg, SW14 SW_Push_45deg, SW15 SW_Push_45deg, SW16 SW_Push_45deg, SW17 SW_Push_45deg, SW18 SW_Push_45deg, SW19 SW_Push_45deg, SW2 SW_Push_45deg, SW20 SW_Push_45deg, SW21 SW_Push_45deg, SW22 SW_Push_45deg, SW23 SW_Push_45deg, SW24 SW_Push_45deg, SW25 SW_Push_45deg, SW26 SW_Push_45deg, SW27 SW_Push_45deg, SW29 SW_Push_45deg, SW3 SW_Push_45deg, SW30 SW_Push_45deg, SW31 SW_Push_45deg, SW32 SW_Push_45deg, SW33 SW_Push_45deg, SW34 SW_Push_45deg, SW36 SW_Push_45deg, SW37 SW_Push_45deg, SW38 SW_Push_45deg, SW39 SW_Push_45deg, SW4 SW_Push_45deg, SW5 SW_Push_45deg, SW6 SW_Push_45deg, SW7 SW_Push_45deg, SW8 SW_Push_45deg, SW9 SW_Push_45deg, U1 nice_nano, U2 nice_nano

Commit message: second update
Parts:
- removed D38, D39: 1N4148, Diode_THT:D_DO-35_SOD27_P7.62mm_Horizontal, symbol Diode:1N4148
- removed SW38, SW39: SW_Push_45deg, symbol Switch:SW_Push_45deg
- removed U2: nice_nano, symbol nicenano:nice_nano
- added D28, D35: 1N4148, Diode_THT:D_DO-35_SOD27_P7.62mm_Horizontal, symbol Diode:1N4148
- added SW28, SW35: SW_Push_45deg, symbol Switch:SW_Push_45deg
- added SW84: SW_Push, symbol Switch:SW_Push
Connections:
- net col_L5: now reaches SW12.1, SW19.1, SW26.1, SW5.1
- net col_L5: now also SW32.1, U1.7 (P0.22); no longer SW33.1
- net col_L1: now reaches SW1.1, SW15.1, SW22.1, SW8.1
- net col_L1: now also SW34.1, U1.1 (TX0/P0.06), SW28.1; no longer SW29.1, SW36.1
- net row_L4: now reaches D22.1 (K), D23.1 (K), D24.1 (K), D25.1 (K), D26.1 (K), D27.1 (K)
- net row_L4: now also U1.13 (NFC1/P0.09)
- net col_L3: now reaches SW10.1, SW17.1, SW24.1, SW3.1
- net col_L3: now also SW30.1, SW36.1, U1.5 (P0.17); no longer SW31.1
- net row_L2: now reaches D10.1 (K), D11.1 (K), D12.1 (K), D13.1 (K), D14.1 (K), D8.1 (K), D9.1 (K)
- net row_L2: now also U1.11 (P1.04)
- net col_L4: now reaches SW11.1, SW18.1, SW25.1, SW4.1
- net col_L4: now also SW31.1, SW37.1, U1.6 (P0.20); no longer SW32.1
- net row_L1: now reaches D1.1 (K), D2.1 (K), D3.1 (K), D4.1 (K), D5.1 (K), D6.1 (K), D7.1 (K)
- net row_L1: now also U1.10 (P0.11)
- net row_L6: now reaches D36.1 (K), D37.1 (K)
- net row_L6: now also D34.1 (K), U1.15 (P1.11), D35.1 (K)
- net row_L3: now reaches U1.12 (P1.06)
- net row_L3: now also D15.1 (K), D16.1 (K), D17.1 (K), D18.1 (K), D19.1 (K), D20.1 (K), D21.1 (K)
- net row_L5: now reaches U1.14 (NFC2/P0.10)
- net row_L5: now also D29.1 (K), D30.1 (K), D31.1 (K), D32.1 (K), D33.1 (K), D28.1 (K)
- net col_L2: now reaches U1.2 (RX1/P0.08)
- net col_L2: now also SW16.1, SW2.1, SW23.1, SW29.1, SW9.1, SW35.1
- net RST_L: now reaches U1.22 (RST)
- net RST_L: now also SW84.1
- net GND_MCU1: now reaches U1.23 (GND)
- net BATIN: now reaches U1.24 (BATIN/P0.04)
- net col_L6: now reaches U1.8 (P0.24)
- net col_L6: now also SW13.1, SW20.1, SW27.1, SW33.1, SW6.1
- net col_L7: now reaches U1.9 (P1.00)
- net col_L7: now also SW14.1, SW21.1, SW7.1
- new net: D28.2 (A), SW28.2
- new net: D35.2 (A), SW35.2
- new net GND: SW84.2
- no-connect marks 0 -> 10
Other:
- moved on the sheet: D1, SW1, U1
